File: eCAD/Bachelor thesis/Main board/Main board.brd (EAGLE design)
At the start: 100 x 98 mm, 111 parts, among them IC1 ESP32-WROOM-32E_M113EH3200PH3Q, IC10 SMS3.3.TCT, IC2 BC660K-GL, IC3 SMS3.3.TCT, IC4 AP9101CK6-ADTRG1, IC5 FDS6898A, IC6 MCP73871-2CCI_ML, IC7 ME6211C33M5G-N, IC8 ME6211C33M5G-N, IC9 SMS3.3.TCT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

Commit message: Misc
Connections:
- net PROG2 renamed PROG3
- net PROG4 renamed PROG1
Changed lines of the file:
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@@
 <wire x1="20.5" y1="48.05" x2="20.5" y2="52.0742625" width="0.2" layer="1"/>
 </signal>
-<signal name="PROG2">
+<signal name="PROG3">
 <contactref element="IC6" pad="12"/>
 <contactref element="R24" pad="1"/>
@@
 <wire x1="22.7" y1="49.9" x2="21.8" y2="49" width="0.2" layer="1"/>
 </signal>
-<signal name="PROG4">
+<signal name="PROG1">
 <contactref element="IC6" pad="13"/>
 <contactref element="R25" pad="1"/>

Commit message: Corrected mistakes
Parts:
- removed C3: 100n, rcl:C0603
- C17: value 100n -> (none)
- R9: value 2k2 -> 470
- moved R3 1.40 mm to (61.2, 51.4)
Connections:
- net GND: now also JP5.1; no longer C3.2, R3.1
- net PSM_EINT: now also JP5.2, R3.1; no longer JP5.1, R3.2
- net RESET_N: no longer C3.1
- net VDD33: now also R3.2; no longer JP5.2
Routing:
- net PSM_EINT: track 78.6 -> 58.4 mm
- net VDD33: track 62.9 -> 64.7 mm, vias 8 -> 9
- net RESET_N: track 67.3 -> 68.2 mm
Changed lines of the file:
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@@
 </layers>
 <board>
-<fusionsync huburn="a.YnVzaW5lc3M6Z21haWwxMjg5Mjg3" projecturn="a.YnVzaW5lc3M6Z21haWwxMjg5Mjg3IzIwMjIxMjE2NTg5ODM1NTUx" f3durn="urn:adsk.wipprod:dm.lineage:cTlje76PRjGCdoz_PzEfoQ" pcbguid="" lastpulledtime="" lastsyncedchangeguid="" latestrevisionid="32a4e163-b02b-4606-8c50-fcb28e7b7cd0" lastsyncedrevisionid="32a4e163-b02b-4606-8c50-fcb28e7b7cd0" lastboardhashguid="d0113ea3-23f0-f7d0-e42b-7ed67bf3e51a" lastpushedtime="2023-04-16T09:40:48Z" linktopcb3d="true"/>
+<fusionsync huburn="a.YnVzaW5lc3M6Z21haWwxMjg5Mjg3" projecturn="a.YnVzaW5lc3M6Z21haWwxMjg5Mjg3IzIwMjIxMjE2NTg5ODM1NTUx" f3durn="urn:adsk.wipprod:dm.lineage:cTlje76PRjGCdoz_PzEfoQ" pcbguid="" lastpulledtime="" lastsyncedchangeguid="" latestrevisionid="85918d6a-9694-4930-9db8-8410fdbd60fd" lastsyncedrevisionid="85918d6a-9694-4930-9db8-8410fdbd60fd" lastboardhashguid="0f75e0a1-0358-cb4b-6328-cdabef2a6fdb" lastpushedtime="2023-05-18T18:45:17Z" linktopcb3d="true"/>
 <plain>
 <wire x1="-1" y1="0" x2="9.8" y2="0" width="0" layer="20"/>
@@
 <attribute name="SPICEPREFIX" value="C" x="122.22" y="99.86" size="1.778" layer="27" rot="R90" display="off"/>
 </element>
-<element name="C17" library="rcl" library_urn="urn:adsk.eagle:library:334" package="C0603" package3d_urn="urn:adsk.eagle:package:23616/2" value="100n" x="30.4" y="58.8" smashed="yes" rot="R270">
+<element name="C17" library="rcl" library_urn="urn:adsk.eagle:library:334" package="C0603" package3d_urn="urn:adsk.eagle:package:23616/2" value="" x="30.4" y="58.8" smashed="yes" rot="R270">
 <attribute name="NAME" x="30.4" y="60.4" size="1.27" layer="25" rot="R90" align="center-left"/>
 <attribute name="POPULARITY" value="73" x="-78.82" y="29.59" size="1.778" layer="27" rot="R270" display="off"/>
@@
 <attribute name="SPICEPREFIX" value="C" x="96.21" y="137.82" size="1.778" layer="28" rot="MR180" display="off"/>
 </element>
-<element name="C3" library="rcl" library_urn="urn:adsk.eagle:library:334" package="C0603" package3d_urn="urn:adsk.eagle:package:23616/2" value="100n" x="74.4" y="55.2" smashed="yes">
-<attribute name="NAME" x="74.4" y="56.2" size="1.27" layer="25" align="bottom-center"/>
-<attribute name="POPULARITY" value="73" x="135.36" y="-54.02" size="1.778" layer="27" display="off"/>
-<attribute name="SPICEPREFIX" value="C" x="135.36" y="-54.02" size="1.778" layer="27" display="off"/>
-</element>
 <element name="C5" library="rcl" library_urn="urn:adsk.eagle:library:334" package="C0603" package3d_urn="urn:adsk.eagle:package:23616/2" value="100n" x="66.46" y="88.91" smashed="yes" rot="R270">
 <attribute name="NAME" x="66.46" y="90.91" size="1.27" layer="25" rot="R90" align="center-left"/>
@@
 <attribute name="VALUE" x="53.66" y="79.835" size="1.27" layer="27" rot="R270"/>
 </element>
-<element name="R9" library="rcl" library_urn="urn:adsk.eagle:library:334" package="R0603" package3d_urn="urn:adsk.eagle:package:23555/3" value="2k2" x="18.4" y="66.8" smashed="yes" rot="R180">
+<element name="R9" library="rcl" library_urn="urn:adsk.eagle:library:334" package="R0603" package3d_urn="urn:adsk.eagle:package:23555/3" value="470" x="18.4" y="66.8" smashed="yes" rot="R180">
 <attribute name="NAME" x="20.4" y="66.8" size="1.27" layer="25" align="center-left"/>
 <attribute name="POPULARITY" value="70" x="3.16" y="188.72" size="1.778" layer="27" rot="R180" display="off"/>
@@
 <attribute name="SPICEPREFIX" value="R" x="159.11" y="144.77" size="1.778" layer="28" rot="MR180" display="off"/>
 </element>
-<element name="R3" library="rcl" library_urn="urn:adsk.eagle:library:334" package="R0603" package3d_urn="urn:adsk.eagle:package:23555/3" value="10k" x="59.8" y="51.4" smashed="yes" rot="R90">
-<attribute name="NAME" x="57.93" y="50.365" size="1.27" layer="25" rot="R90" align="center-left"/>
-<attribute name="POPULARITY" value="70" x="175.37" y="159.35" size="1.778" layer="27" rot="R90" display="off"/>
-<attribute name="SPICEPREFIX" value="R" x="175.37" y="159.35" size="1.778" layer="27" rot="R90" display="off"/>
+<element name="R3" library="rcl" library_urn="urn:adsk.eagle:library:334" package="R0603" package3d_urn="urn:adsk.eagle:package:23555/3" value="10k" x="61.2" y="51.4" smashed="yes" rot="R90">
+<attribute name="NAME" x="59.33" y="50.365" size="1.27" layer="25" rot="R90" align="center-left"/>
+<attribute name="POPULARITY" value="70" x="176.77" y="159.35" size="1.778" layer="27" rot="R90" display="off"/>
+<attribute name="SPICEPREFIX" value="R" x="176.77" y="159.35" size="1.778" layer="27" rot="R90" display="off"/>
 </element>
 <element name="R4" library="rcl" library_urn="urn:adsk.eagle:library:334" package="R0603" package3d_urn="urn:adsk.eagle:package:23555/3" value="10k" x="15.2" y="77" smashed="yes" rot="R270">
@@
 <contactref element="IC1" pad="15"/>
 <contactref element="JP6" pad="4"/>
-<contactref element="R3" pad="1"/>
 <contactref element="JP7" pad="4"/>
-<contactref element="C3" pad="2"/>
 <contactref element="JP3" pad="2"/>
 <contactref element="JP4" pad="2"/>
@@
 <via x="39.8" y="30.6" extent="1-16" drill="0.3" diameter="0.3"/>
 <via x="75.26" y="33.52" extent="1-16" drill="0.3" diameter="0.3"/>
-<via x="76.3524" y="55.1746" extent="1-16" drill="0.3" diameter="0.3"/>
+<via x="75.9524" y="57.3746" extent="1-16" drill="0.3" diameter="0.3"/>
 <via x="90.0762" y="50.2254" extent="1-16" drill="0.3" diameter="0.3"/>
 <via x="66.45" y="90.89" extent="1-16" drill="0.3" diameter="0.7"/>
@@
 <via x="64.021" y="27.9568" extent="1-16" drill="0.3" diameter="0.3"/>
 <via x="62.77" y="40.12" extent="1-16" drill="0.3" diameter="0.3"/>
-<via x="59.4" y="49.6" extent="1-16" drill="0.3" diameter="0.3"/>
+<via x="59.4" y="48.6" extent="1-16" drill="0.3" diameter="0.3"/>
 <via x="58.2134" y="34.8292" extent="1-16" drill="0.3" diameter="0.3"/>
 <via x="90" y="80.2" extent="1-16" drill="0.3" diameter="0.5"/>
 <via x="89.2" y="71.6" extent="1-16" drill="0.3" diameter="0.5"/>
 <via x="67.77" y="80.42" extent="1-16" drill="0.35"/>
+<contactref element="JP5" pad="1"/>
 </signal>
 <signal name="ESP_BOOT">
@@
 <contactref element="C4" pad="2"/>
 <contactref element="JP6" pad="1"/>
-<contactref element="JP5" pad="2"/>
 <contactref element="JP7" pad="1"/>
 <contactref element="C14" pad="+"/>
@@
 <wire x1="49.4" y1="91" x2="48.8" y2="90.4" width="1" layer="1"/>
 <wire x1="80.45" y1="55.2" x2="81.4" y2="55.2" width="1" layer="1"/>
+<contactref element="R3" pad="2"/>
+<via x="59.4" y="52.2" extent="1-16" drill="0.35"/>
+<wire x1="59.4" y1="52.2" x2="59.45" y2="52.25" width="0.5" layer="1"/>
+<wire x1="59.45" y1="52.25" x2="61.2" y2="52.25" width="0.5" layer="1"/>
 </signal>
 <signal name="VOL_SENS">
@@
 <signal name="RESET_N">
 <contactref element="JP3" pad="1"/>
-<contactref element="C3" pad="1"/>
 <contactref element="Q1" pad="3"/>
 <contactref element="C17" pad="1"/>
@@
 <wire x1="39.84" y1="68.6" x2="39.84" y2="68.64" width="0.2" layer="1"/>
 <wire x1="37.8" y1="66" x2="39.84" y2="68.04" width="0.2" layer="1"/>
-<wire x1="73.55" y1="55.2" x2="73.55" y2="53.32" width="0.5" layer="1"/>
 <wire x1="73.55" y1="53.32" x2="74.2" y2="52.67" width="0.5" layer="1"/>
-<wire x1="73.55" y1="55.2" x2="72.4" y2="56.35" width="0.5" layer="1"/>
-<wire x1="72.4" y1="56.35" x2="72.4" y2="63.2" width="0.5" layer="1"/>
 <wire x1="71.389" y1="64.211" x2="44.7022875" y2="64.211" width="0.5" layer="1"/>
 <wire x1="44.7022875" y1="64.211" x2="42.5132875" y2="66.4" width="0.5" layer="1"/>
@@
 <wire x1="39.8" y1="67.2" x2="39.8" y2="68.56" width="0.5" layer="1"/>
 <wire x1="39.8" y1="68.56" x2="39.84" y2="68.6" width="0.5" layer="1"/>
-<wire x1="72.4" y1="63.2" x2="71.389" y2="64.211" width="0.5" layer="1"/>
+<wire x1="71.389" y1="64.211" x2="72.4" y2="63.2" width="0.5" layer="1"/>
 <wire x1="42.5132875" y1="66.4" x2="40.6" y2="66.4" width="0.5" layer="1"/>
+<wire x1="72.4" y1="54.47" x2="74.2" y2="52.67" width="0.5" layer="1"/>
+<wire x1="72.4" y1="63.2" x2="72.4" y2="54.47" width="0.5" layer="1"/>
 </signal>
 <signal name="BOOT">
@@
 </signal>
 <signal name="PSM_EINT">
-<contactref element="R3" pad="2"/>
-<contactref element="JP5" pad="1"/>
 <contactref element="IC1" pad="29"/>
 <contactref element="IC2" pad="19"/>
-<wire x1="59.8" y1="52.25" x2="60.22" y2="52.67" width="0.5" layer="1"/>
-<wire x1="60.22" y1="52.67" x2="64.4" y2="52.67" width="0.5" layer="1"/>
-<wire x1="64.4" y1="52.67" x2="64.4" y2="62.557" width="0.5" layer="1"/>
 <wire x1="64.4" y1="62.557" x2="64" y2="62.957" width="0.5" layer="1"/>
 <wire x1="64" y1="62.957" x2="46.757" y2="62.957" width="0.5" layer="1"/>
@@
 <wire x1="82.7" y1="78.1" x2="80" y2="75.4" width="0.5" layer="16"/>
 <wire x1="78.2" y1="75.4" x2="64.4" y2="61.6" width="0.5" layer="16"/>
-<wire x1="64.4" y1="61.6" x2="64.4" y2="52.67" width="0.5" layer="16"/>
 <wire x1="80" y1="75.4" x2="78.2" y2="75.4" width="0.5" layer="16"/>
+<contactref element="JP5" pad="2"/>
+<contactref element="R3" pad="1"/>
+<wire x1="61.2" y1="50.55" x2="63.25" y2="50.55" width="0.5" layer="1"/>
+<wire x1="63.67" y1="50.13" x2="64.4" y2="50.13" width="0.5" layer="1"/>
+<wire x1="63.25" y1="50.55" x2="63.67" y2="50.13" width="0.5" layer="1"/>
+<wire x1="64.4" y1="62.557" x2="64.4" y2="61.6" width="0" layer="19" extent="1-16"/>
+<wire x1="64.4" y1="50.13" x2="64.4" y2="61.6" width="0" layer="19" extent="16-16"/>
 </signal>
 <signal name="NETLIGHT">
